Commit message: Acquire Hint State

File: exp_assignment3/urdf/sherlock.urdf (robot description, URDF)
Before this commit: robot sherlock, 12 links, 11 joints
Joints:
- joint arm_base_to_base: limit lower=-3.14 upper=3.14 effort=1000.0 velocity=0.2 -> lower=-3.14 upper=3.14 effort=1000.0 velocity=0.5
- joint arm_joint_01: limit lower=-1.57 upper=1.57 effort=1000.0 velocity=0.2 -> lower=-1.57 upper=1.57 effort=1000.0 velocity=0.5
- joint arm_joint_02: limit lower=-3 upper=3 effort=1000.0 velocity=0.2 -> lower=-3 upper=3 effort=1000.0 velocity=0.5
- joint arm_joint_03: limit lower=-3 upper=3 effort=1000.0 velocity=0.2 -> lower=-3 upper=3 effort=1000.0 velocity=0.5

Commit message: Restored initial joints velocities

File: exp_assignment3/urdf/sherlock.urdf (robot description, URDF)
Before this commit: robot sherlock, 12 links, 11 joints
Joints:
- joint arm_base_to_base: limit lower=-3.14 upper=3.14 effort=1000.0 velocity=0.5 -> lower=-3.14 upper=3.14 effort=1000.0 velocity=0.2
- joint arm_joint_01: limit lower=-1.57 upper=1.57 effort=1000.0 velocity=0.5 -> lower=-1.57 upper=1.57 effort=1000.0 velocity=0.2
- joint arm_joint_02: limit lower=-3 upper=3 effort=1000.0 velocity=0.5 -> lower=-3 upper=3 effort=1000.0 velocity=0.2
- joint arm_joint_03: limit lower=-3 upper=3 effort=1000.0 velocity=0.5 -> lower=-3 upper=3 effort=1000.0 velocity=0.2
- joint arm_joint_04: limit lower=-1.57 upper=1.57 effort=1000.0 velocity=0.5 -> lower=-1.57 upper=1.57 effort=1000.0 velocity=0.2

Commit message: Move Base Problem solved

File: exp_assignment3/urdf/sherlock.urdf (robot description, URDF)
Before this commit: robot sherlock, 12 links, 11 joints
Joints:
- joint camera_joint: origin xyz=0 0 0.05 rpy=0 0 0 -> xyz=0 0 0.05 rpy=0 0 1.57

Commit message: Adjustments

File: exp_assignment3/urdf/sherlock.urdf (robot description, URDF)
Before this commit: robot sherlock, 12 links, 11 joints
Joints:
- joint arm_base_to_base: limit lower=-3.14 upper=3.14 effort=1000.0 velocity=0.2 -> lower=-3.14 upper=3.14 effort=1000.0 velocity=.5
- joint arm_joint_01: limit lower=-1.57 upper=1.57 effort=1000.0 velocity=0.2 -> lower=-1.57 upper=1.57 effort=1000.0 velocity=.5
- joint arm_joint_02: limit lower=-3 upper=3 effort=1000.0 velocity=0.2 -> lower=-3 upper=3 effort=1000.0 velocity=.5
- joint arm_joint_03: limit lower=-3 upper=3 effort=1000.0 velocity=0.2 -> lower=-3 upper=3 effort=1000.0 velocity=.5
- joint arm_joint_04: limit lower=-1.57 upper=1.57 effort=1000.0 velocity=0.2 -> lower=-1.57 upper=1.57 effort=1000.0 velocity=.5
